File: qwiic-hat.kicad_sch (KiCad schematic)
At the start: 4 parts, among them J1 Conn_02x20_Odd_Even, J2 Conn_01x04_Male, J3 Conn_01x04_Male, J4 Conn_01x03_Pin

Commit message: cleanup sheets
Other:
- company: (none) -> Karolis Stasaitis (carlossless.io)
- moved on the sheet: J1, J2, J3, J4
